File: V1/esp-poe-4rl-V1.kicad_sch (KiCad schematic)
At the start: 56 parts, among them J1 USB_C_Receptacle_USB2.0, J3 RJ45 JACK, Q1 UMH3N, Q3 WPM2015-3/TR, Q4 LMUN2211LT1G, SW1 RESET, U1 CH340K, U2 ESP32-WROOM-32UE-N16, U3 LAN8710A

Commit message: Under development.
Changed lines of the file:
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@@
 	)
 	(junction
+		(at 227.965 67.31)
+		(diameter 0)
+		(color 0 0 0 0)
+	)
+	(junction
 		(at 367.03 85.09)
 		(diameter 0)
@@
 	)
 	(junction
-		(at 227.965 67.31)
-		(diameter 0)
-		(color 0 0 0 0)
-	)
-	(junction
 		(at 21.59 90.17)
 		(diameter 0)
@@
 	(wire
 		(pts
+			(xy 223.52 67.31) (xy 227.965 67.31)
+		)
+		(stroke
+			(width 0)
+			(type default)
+		)
+	)
+	(wire
+		(pts
 			(xy 123.19 76.2) (xy 129.54 76.2)
 		)
@@
 	(wire
 		(pts
+			(xy 220.98 74.93) (xy 220.98 60.325)
+		)
+		(stroke
+			(width 0)
+			(type default)
+		)
+	)
+	(wire
+		(pts
 			(xy 210.82 36.83) (xy 210.82 64.77)
 		)
@@
 	(wire
 		(pts
-			(xy 218.44 69.85) (xy 218.44 56.515)
-		)
-		(stroke
-			(width 0)
-			(type default)
-		)
-	)
-	(wire
-		(pts
 			(xy 283.21 31.75) (xy 283.21 34.29)
 		)
@@
 	(wire
 		(pts
-			(xy 220.98 61.595) (xy 230.505 61.595)
-		)
-		(stroke
-			(width 0)
-			(type default)
-		)
-	)
-	(wire
-		(pts
 			(xy 158.75 214.63) (xy 158.75 209.55)
 		)
@@
 		)
 	)
+	(wire
+		(pts
+			(xy 227.965 67.31) (xy 227.965 68.58)
+		)
+		(stroke
+			(width 0)
+			(type default)
+		)
+	)
 	(polyline
 		(pts
@@
 	(wire
 		(pts
+			(xy 227.965 76.2) (xy 227.965 77.47)
+		)
+		(stroke
+			(width 0)
+			(type default)
+		)
+	)
+	(wire
+		(pts
 			(xy 283.21 41.91) (xy 283.21 95.25)
 		)
@@
 	(wire
 		(pts
+			(xy 223.52 80.01) (xy 223.52 67.31)
+		)
+		(stroke
+			(width 0)
+			(type default)
+		)
+	)
+	(wire
+		(pts
 			(xy 283.21 95.25) (xy 303.53 95.25)
 		)
@@
 	(wire
 		(pts
-			(xy 227.965 67.31) (xy 230.505 67.31)
-		)
-		(stroke
-			(width 0)
-			(type default)
-		)
-	)
-	(wire
-		(pts
 			(xy 383.54 125.73) (xy 388.62 125.73)
 		)
@@
 	(wire
 		(pts
-			(xy 218.44 56.515) (xy 230.505 56.515)
+			(xy 372.11 132.08) (xy 375.92 132.08)
 		)
 		(stroke
@@
 	(wire
 		(pts
-			(xy 372.11 132.08) (xy 375.92 132.08)
+			(xy 218.44 69.85) (xy 218.44 55.245)
 		)
 		(stroke
@@
 	(wire
 		(pts
-			(xy 227.965 67.31) (xy 227.965 68.58)
+			(xy 163.83 60.96) (xy 163.83 34.29)
 		)
 		(stroke
@@
 	(wire
 		(pts
-			(xy 163.83 60.96) (xy 163.83 34.29)
+			(xy 274.32 129.54) (xy 274.32 132.08)
 		)
 		(stroke
@@
 	(wire
 		(pts
-			(xy 274.32 129.54) (xy 274.32 132.08)
+			(xy 227.965 67.31) (xy 230.505 67.31)
 		)
 		(stroke
@@
 	(wire
 		(pts
-			(xy 223.52 67.31) (xy 227.965 67.31)
-		)
-		(stroke
-			(width 0)
-			(type default)
-		)
-	)
-	(wire
-		(pts
-			(xy 227.965 76.2) (xy 227.965 77.47)
-		)
-		(stroke
-			(width 0)
-			(type default)
-		)
-	)
-	(wire
-		(pts
 			(xy 402.59 106.68) (xy 402.59 82.55)
 		)
@@
 	(wire
 		(pts
+			(xy 218.44 55.245) (xy 230.505 55.245)
+		)
+		(stroke
+			(width 0)
+			(type default)
+		)
+	)
+	(wire
+		(pts
 			(xy 336.55 195.58) (xy 336.55 200.66)
 		)
@@
 	(wire
 		(pts
-			(xy 220.98 74.93) (xy 220.98 61.595)
-		)
-		(stroke
-			(width 0)
-			(type default)
-		)
-	)
-	(wire
-		(pts
 			(xy 204.47 113.03) (xy 264.16 113.03)
 		)
@@
 	(wire
 		(pts
+			(xy 220.98 60.325) (xy 230.505 60.325)
+		)
+		(stroke
+			(width 0)
+			(type default)
+		)
+	)
+	(wire
+		(pts
 			(xy 140.97 100.33) (xy 140.97 102.87)
 		)
@@
 	(wire
 		(pts
-			(xy 223.52 80.01) (xy 223.52 67.31)
-		)
-		(stroke
-			(width 0)
-			(type default)
-		)
-	)
-	(wire
-		(pts
 			(xy 123.19 60.96) (xy 163.83 60.96)
 		)
@@
 	(global_label "OUT3"
 		(shape output)
-		(at 230.505 56.515 0)
+		(at 230.505 55.245 0)
 		(fields_autoplaced yes)
 		(effects
@@
 		)
 		(property "Intersheetrefs" "${INTERSHEET_REFS}"
-			(at 237.6741 56.515 0)
+			(at 237.6741 55.245 0)
 			(hide yes)
 			(show_name no)
@@
 	(global_label "OUT4"
 		(shape output)
-		(at 230.505 61.595 0)
+		(at 230.505 60.325 0)
 		(fields_autoplaced yes)
 		(effects
@@
 		)
 		(property "Intersheetrefs" "${INTERSHEET_REFS}"
-			(at 237.6741 61.595 0)
+			(at 237.6741 60.325 0)
 			(hide yes)
 			(show_name no)

Commit message: Development
Parts:
- renumbered J3 to J2, Q3 to Q2, Q4 to Q3, R25 to R21, R24 to R22, R28 to R23, R26 to R24
Changed lines of the file:
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@@
 		(dnp no)
 		(fields_autoplaced yes)
-		(property "Reference" "R24"
+		(property "Reference" "R22"
 			(at 364.49 223.5199 0)
 			(show_name no)
@@
 			(project "esp-poe-4rl-V1"
 				(path "/2bc5a21a-1d79-419d-a592-6852cc07b00a"
-					(reference "R24")
+					(reference "R22")
 					(unit 1)
 				)
@@
 		(dnp no)
 		(fields_autoplaced yes)
-		(property "Reference" "#PWR048"
+		(property "Reference" "#PWR043"
 			(at 203.2 227.33 0)
 			(hide yes)
@@
 			(project "esp-poe-4rl-V1"
 				(path "/2bc5a21a-1d79-419d-a592-6852cc07b00a"
-					(reference "#PWR048")
+					(reference "#PWR043")
 					(unit 1)
 				)
@@
 		(in_pos_files yes)
 		(dnp no)
-		(property "Reference" "#PWR042"
+		(property "Reference" "#PWR041"
 			(at 203.2 210.82 0)
 			(hide yes)
@@
 			(project "esp-poe-4rl-V1"
 				(path "/2bc5a21a-1d79-419d-a592-6852cc07b00a"
-					(reference "#PWR042")
+					(reference "#PWR041")
 					(unit 1)
 				)
@@
 		(in_pos_files yes)
 		(dnp no)
-		(property "Reference" "#PWR052"
+		(property "Reference" "#PWR049"
 			(at 342.9 251.46 0)
 			(hide yes)
@@
 			(project "esp-poe-4rl-V1"
 				(path "/2bc5a21a-1d79-419d-a592-6852cc07b00a"
-					(reference "#PWR052")
+					(reference "#PWR049")
 					(unit 1)
 				)
@@
 		(in_pos_files yes)
 		(dnp no)
-		(property "Reference" "#PWR041"
+		(property "Reference" "#PWR040"
 			(at 158.75 210.82 0)
 			(hide yes)
@@
 			(project "esp-poe-4rl-V1"
 				(path "/2bc5a21a-1d79-419d-a592-6852cc07b00a"
-					(reference "#PWR041")
+					(reference "#PWR040")
 					(unit 1)
 				)
@@
 		(dnp no)
 		(fields_autoplaced yes)
-		(property "Reference" "#PWR050"
+		(property "Reference" "#PWR045"
 			(at 242.57 227.33 0)
 			(hide yes)
@@
 			(project "esp-poe-4rl-V1"
 				(path "/2bc5a21a-1d79-419d-a592-6852cc07b00a"
-					(reference "#PWR050")
+					(reference "#PWR045")
 					(unit 1)
 				)
@@
 		(in_pos_files yes)
 		(dnp no)
-		(property "Reference" "Q3"
+		(property "Reference" "Q2"
 			(at 187.96 200.66 90)
 			(show_name no)
@@
 			(project "esp-poe-4rl-V1"
 				(path "/2bc5a21a-1d79-419d-a592-6852cc07b00a"
-					(reference "Q3")
+					(reference "Q2")
 					(unit 1)
 				)
@@
 		(dnp no)
 		(fields_autoplaced yes)
-		(property "Reference" "R26"
+		(property "Reference" "R24"
 			(at 345.44 236.2199 0)
 			(show_name no)
@@
 			(project "esp-poe-4rl-V1"
 				(path "/2bc5a21a-1d79-419d-a592-6852cc07b00a"
-					(reference "R26")
+					(reference "R24")
 					(unit 1)
 				)
@@
 		(in_pos_files yes)
 		(dnp no)
-		(property "Reference" "#PWR043"
+		(property "Reference" "#PWR042"
 			(at 251.46 210.82 0)
 			(hide yes)
@@
 			(project "esp-poe-4rl-V1"
 				(path "/2bc5a21a-1d79-419d-a592-6852cc07b00a"
-					(reference "#PWR043")
+					(reference "#PWR042")
 					(unit 1)
 				)
@@
 		(dnp no)
 		(fields_autoplaced yes)
-		(property "Reference" "#PWR049"
+		(property "Reference" "#PWR044"
 			(at 220.98 227.33 0)
 			(hide yes)
@@
 			(project "esp-poe-4rl-V1"
 				(path "/2bc5a21a-1d79-419d-a592-6852cc07b00a"
-					(reference "#PWR049")
+					(reference "#PWR044")
 					(unit 1)
 				)
@@
 		(dnp no)
 		(fields_autoplaced yes)
-		(property "Reference" "#PWR053"
+		(property "Reference" "#PWR047"
 			(at 224.79 246.38 0)
 			(hide yes)
@@
 			(project "esp-poe-4rl-V1"
 				(path "/2bc5a21a-1d79-419d-a592-6852cc07b00a"
-					(reference "#PWR053")
+					(reference "#PWR047")
 					(unit 1)
 				)
@@
 		(dnp no)
 		(fields_autoplaced yes)
-		(property "Reference" "R25"
+		(property "Reference" "R21"
 			(at 179.07 215.265 0)
 			(show_name no)
@@
 			(project "esp-poe-4rl-V1"
 				(path "/2bc5a21a-1d79-419d-a592-6852cc07b00a"
-					(reference "R25")
+					(reference "R21")
 					(unit 1)
 				)
@@
 		(dnp no)
 		(fields_autoplaced yes)
-		(property "Reference" "R28"
+		(property "Reference" "R23"
 			(at 195.58 229.235 0)
 			(show_name no)
@@
 			(project "esp-poe-4rl-V1"
 				(path "/2bc5a21a-1d79-419d-a592-6852cc07b00a"
-					(reference "R28")
+					(reference "R23")
 					(unit 1)
 				)
@@
 		(in_pos_files yes)
 		(dnp no)
-		(property "Reference" "Q4"
+		(property "Reference" "Q3"
 			(at 218.44 245.11 90)
 			(show_name no)
@@
 			(project "esp-poe-4rl-V1"
 				(path "/2bc5a21a-1d79-419d-a592-6852cc07b00a"
-					(reference "Q4")
+					(reference "Q3")
 					(unit 1)
 				)
@@
 		(in_pos_files yes)
 		(dnp no)
-		(property "Reference" "#PWR051"
+		(property "Reference" "#PWR048"
 			(at 287.02 246.38 0)
 			(hide yes)
@@
 			(project "esp-poe-4rl-V1"
 				(path "/2bc5a21a-1d79-419d-a592-6852cc07b00a"
-					(reference "#PWR051")
+					(reference "#PWR048")
 					(unit 1)
 				)
@@
 		(in_pos_files yes)
 		(dnp no)
-		(property "Reference" "#PWR045"
+		(property "Reference" "#PWR046"
 			(at 347.98 232.41 0)
 			(hide yes)
@@
 			(project "esp-poe-4rl-V1"
 				(path "/2bc5a21a-1d79-419d-a592-6852cc07b00a"
-					(reference "#PWR045")
+					(reference "#PWR046")
 					(unit 1)
 				)
@@
 		(in_pos_files yes)
 		(dnp no)
-		(property "Reference" "#PWR040"
+		(property "Reference" "#PWR039"
 			(at 336.55 207.01 0)
 			(hide yes)
@@
 			(project "esp-poe-4rl-V1"
 				(path "/2bc5a21a-1d79-419d-a592-6852cc07b00a"
-					(reference "#PWR040")
+					(reference "#PWR039")
 					(unit 1)
 				)
@@
 		(dnp no)
 		(fields_autoplaced yes)
-		(property "Reference" "J3"
+		(property "Reference" "J2"
 			(at 313.69 151.13 0)
 			(show_name no)
@@
 			(project "esp-poe-4rl-V1"
 				(path "/2bc5a21a-1d79-419d-a592-6852cc07b00a"
-					(reference "J3")
+					(reference "J2")
 					(unit 1)
 				)

Commit message: V1.0.0
Connections:
- net OUT3: now also U2.9 (IO33); no longer U2.24 (IO2)
- net OUT4: now also U2.8 (IO32); no longer U2.26 (IO4)
Other:
- moved on the sheet: R10
