File: V1/esp-poe-4rl-V1-power.kicad_sch (KiCad schematic)
At the start: 31 parts, among them U4 TPS2376DDAR-H, U5 TX4138, U6 SY8089A1AAC

Commit message: Development
Parts:
- renumbered D7 to D3, D8 to D4, D9 to D5, D10 to D6, D11 to D7, R31 to R25, R32 to R26, R33 to R27, R34 to R28, R35 to R29, R36 to R30, R37 to R31, R38 to R32, R39 to R33, R40 to R34, R41 to R35, R42 to R36, R43 to R37

Commit message: Adjusting traces width.
Other:
- title: ESP 2x Relay Output Module with PoE -> ESP 4x Relay Output Module with PoE
Changed lines of the file:
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@@
 	(paper "A4")
 	(title_block
-		(title "ESP 2x Relay Output Module with PoE")
-		(date "2026-01-29")
+		(title "ESP 4x Relay Output Module with PoE")
+		(date "2026-06-10")
 		(rev "V1.0")
 	)
