File: V1/esp-poe-4rl-v1-outputs.kicad_sch (KiCad schematic)
At the start: 32 parts, among them J2 Conn_01x03, J4 Conn_01x03, J5 Conn_01x03, J6 Conn_01x03, K1 G5Q-14-DC5, K2 G5Q-14-DC5, K3 G5Q-14-DC5, K4 G5Q-14-DC5, Q2 MMBT2222A, Q5 MMBT2222A, Q6 MMBT2222A, Q7 MMBT2222A

Commit message: Under development.
Parts:
- J2, J4, J5, J6: value Conn_01x03 -> 250-203; footprint (none) -> Tales:TerminalBlock_Wago_250-203_1x03_P3.5mm_45Degree; JLCPCB BOM (none) -> 1; LCSC Part # (none) -> C2765062; Mfr (none) -> Wago; Mfr PN (none) -> 250-203; Technology (none) -> Spring Cage; Vendor (none) -> JLCPCB; Vendor PN (none) -> C2765062
- K1, K2, K3, K4: JLCPCB BOM (none) -> 1; LCSC Part # (none) -> C397241; Mfr (none) -> Omron; Mfr PN (none) -> G5Q-14-DC5; Technology (none) -> SPDT; Vendor (none) -> JLCPCB; Vendor PN (none) -> C397241
Other:
- moved on the sheet: D14

Commit message: Development
Parts:
- removed J2, J4, J5, J6: 250-203, Tales:TerminalBlock_Wago_250-203_1x03_P3.5mm_45Degree, symbol Connector_Generic:Conn_01x03
- removed K1, K2, K3, K4: G5Q-14-DC5, Relay_THT:Relay_SPDT_Omron-G5Q-1, symbol Relay:G5Q-1
- added J3, J4, J5, J6: 250-202, Tales:TerminalBlock_Wago_250-202_1x02_P3.5mm_45Degree, symbol Connector_Generic:Conn_01x02
- added K1, K2, K3, K4: G5NB-1A-E-DC5, Tales:Relay_SPST_Omron_G5NB-1A, symbol Tales:G5NB-1A
- renumbered D4 to D10, D12 to D11, D5 to D12, D15 to D13, D6 to D14, D13 to D15, D3 to D8, D14 to D9, Q2 to Q4, Q6 to Q5, Q5 to Q6, R21 to R38, R48 to R39, R22 to R40, R46 to R41, R23 to R42, R44 to R43, R27 to R44, R49 to R45, R29 to R46, R30 to R48, R45 to R49
Connections:
- net +5V: now also K1.1, K2.1, K3.1, K4.1
- net OUT1BJT: no longer Q5.1 (B), R41.1
- net OUT1CMD: now also K1.4
- net OUT1LN: now also J3.1 (Pin_1), K1.2
- net OUT1ON: no longer D11.2 (A), R39.2
- net OUT2: now also R41.2, R43.1; no longer R46.2, R48.1
- net OUT2BJT: now also Q5.1 (B), R41.1; no longer Q6.1 (B), Q7.1 (B), R46.1, R47.1
- net OUT2CMD: now also D11.1 (K), D9.2 (A), Q5.3 (C), K2.4; no longer D12.2 (A), D14.1 (K), Q6.3 (C)
- net OUT2LN: now also J4.1 (Pin_1), K2.2
- net OUT2ON: now also D11.2 (A), R39.2; no longer D14.2 (A), D15.2 (A), R44.2, R45.2
- net OUT3: now also R46.2, R48.1; no longer R41.2, R43.1
- net OUT3CMD: now also D12.2 (A), D14.1 (K), Q6.3 (C), K3.4; no longer D11.1 (K), D9.2 (A), Q5.3 (C)
- net OUT3LN: now also J5.1 (Pin_1), K3.2
- net OUT4LN: now also J6.1 (Pin_1), K4.2
- net OUT24MD renamed OUT4CMD
- net OUT4CMD: now also K4.4
- new net OUT1LD: J3.2 (Pin_2), K1.3
- new net OUT2LD: J4.2 (Pin_2), K2.3
- new net OUT3BJT: Q6.1 (B), R46.1
- new net OUT3LD: J5.2 (Pin_2), K3.3
- new net OUT3ON: D14.2 (A), R44.2
- new net OUT4BJT: Q7.1 (B), R47.1
- new net OUT4LD: J6.2 (Pin_2), K4.3
- new net OUT4ON: D15.2 (A), R45.2
Other:
- moved on the sheet: D11, D13, D15, D9, Q5, Q7, R39, R41, R43, R45, R47, R49

Commit message: V1.0.0
Connections:
- net OUT1LD: now also K1.2; no longer K1.3
- net OUT1LN: now also K1.3; no longer K1.2
- net OUT2LD: now also K2.2; no longer K2.3
- net OUT2LN: now also K2.3; no longer K2.2
- net OUT3LD: now also K3.2; no longer K3.3
- net OUT3LN: now also K3.3; no longer K3.2
- net OUT4LD: now also K4.2; no longer K4.3
- net OUT4LN: now also K4.3; no longer K4.2
Other:
- moved on the sheet: J3, J4, J5, J6

Commit message: Adjusting traces width.
Other:
- title: (none) -> ESP 4x Relay Output Module with PoE
Changed lines of the file:
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@@
 	(paper "A4")
 	(title_block
+		(title "ESP 4x Relay Output Module with PoE")
+		(date "2026-06-10")
 		(rev "V1.0")
 	)
