File: V1/eumesmo-poe-4rl-v1-outputs.kicad_sch (KiCad schematic)
At the start: 32 parts, among them J3 250-202, J4 250-202, J5 250-202, J6 250-202, K1 G5NB-1A-E-DC5, K2 G5NB-1A-E-DC5, K3 G5NB-1A-E-DC5, K4 G5NB-1A-E-DC5, Q4 MMBT2222A, Q5 MMBT2222A, Q6 MMBT2222A, Q7 MMBT2222A

Commit message: Renamed all files to align with eumesmo branding.
Other:
- title: ESP 4x Relay Output Module with PoE -> eumesmo 4x Relay Output Module with PoE
Changed lines of the file:
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@@
 	(paper "A4")
 	(title_block
-		(title "ESP 4x Relay Output Module with PoE")
-		(date "2026-06-10")
+		(title "eumesmo 4x Relay Output Module with PoE")
+		(date "2026-06-16")
 		(rev "V1.0")
 	)
@@
 		)
 		(instances
-			(project "esp-poe-4rl-V1"
+			(project "eumesmo-poe-4rl-v1"
 				(path "/2bc5a21a-1d79-419d-a592-6852cc07b00a/774cc362-9cfe-4197-8571-7d1b1ef33e48"
 					(reference "K2")
@@
 		)
 		(instances
-			(project "esp-poe-4rl-V1"
+			(project "eumesmo-poe-4rl-v1"
 				(path "/2bc5a21a-1d79-419d-a592-6852cc07b00a/774cc362-9cfe-4197-8571-7d1b1ef33e48"
 					(reference "R38")
@@
 		)
 		(instances
-			(project "esp-poe-4rl-V1"
+			(project "eumesmo-poe-4rl-v1"
 				(path "/2bc5a21a-1d79-419d-a592-6852cc07b00a/774cc362-9cfe-4197-8571-7d1b1ef33e48"
 					(reference "K4")
@@
 		)
 		(instances
-			(project "esp-poe-4rl-V1"
+			(project "eumesmo-poe-4rl-v1"
 				(path "/2bc5a21a-1d79-419d-a592-6852cc07b00a/774cc362-9cfe-4197-8571-7d1b1ef33e48"
 					(reference "R41")
@@
 		)
 		(instances
-			(project "esp-poe-4rl-V1"
+			(project "eumesmo-poe-4rl-v1"
 				(path "/2bc5a21a-1d79-419d-a592-6852cc07b00a/774cc362-9cfe-4197-8571-7d1b1ef33e48"
 					(reference "R43")
@@
 		)
 		(instances
-			(project "esp-poe-4rl-V1"
+			(project "eumesmo-poe-4rl-v1"
 				(path "/2bc5a21a-1d79-419d-a592-6852cc07b00a/774cc362-9cfe-4197-8571-7d1b1ef33e48"
 					(reference "D10")
@@
 		)
 		(instances
-			(project "esp-poe-4rl-V1"
+			(project "eumesmo-poe-4rl-v1"
 				(path "/2bc5a21a-1d79-419d-a592-6852cc07b00a/774cc362-9cfe-4197-8571-7d1b1ef33e48"
 					(reference "D12")
@@
 		)
 		(instances
-			(project "esp-poe-4rl-V1"
+			(project "eumesmo-poe-4rl-v1"
 				(path "/2bc5a21a-1d79-419d-a592-6852cc07b00a/774cc362-9cfe-4197-8571-7d1b1ef33e48"
 					(reference "R49")
@@
 		)
 		(instances
-			(project "esp-poe-4rl-V1"
+			(project "eumesmo-poe-4rl-v1"
 				(path "/2bc5a21a-1d79-419d-a592-6852cc07b00a/774cc362-9cfe-4197-8571-7d1b1ef33e48"
 					(reference "D11")
@@
 		)
 		(instances
-			(project "esp-poe-4rl-V1"
+			(project "eumesmo-poe-4rl-v1"
 				(path "/2bc5a21a-1d79-419d-a592-6852cc07b00a/774cc362-9cfe-4197-8571-7d1b1ef33e48"
 					(reference "D15")
@@
 		)
 		(instances
-			(project "esp-poe-4rl-V1"
+			(project "eumesmo-poe-4rl-v1"
 				(path "/2bc5a21a-1d79-419d-a592-6852cc07b00a/774cc362-9cfe-4197-8571-7d1b1ef33e48"
 					(reference "D8")
@@
 		)
 		(instances
-			(project "esp-poe-4rl-V1"
+			(project "eumesmo-poe-4rl-v1"
 				(path "/2bc5a21a-1d79-419d-a592-6852cc07b00a/774cc362-9cfe-4197-8571-7d1b1ef33e48"
 					(reference "#PWR074")
@@
 		)
 		(instances
-			(project "esp-poe-4rl-V1"
+			(project "eumesmo-poe-4rl-v1"
 				(path "/2bc5a21a-1d79-419d-a592-6852cc07b00a/774cc362-9cfe-4197-8571-7d1b1ef33e48"
 					(reference "R42")
@@
 		)
 		(instances
-			(project "esp-poe-4rl-V1"
+			(project "eumesmo-poe-4rl-v1"
 				(path "/2bc5a21a-1d79-419d-a592-6852cc07b00a/774cc362-9cfe-4197-8571-7d1b1ef33e48"
 					(reference "#PWR065")
@@
 		)
 		(instances
-			(project "esp-poe-4rl-V1"
+			(project "eumesmo-poe-4rl-v1"
 				(path "/2bc5a21a-1d79-419d-a592-6852cc07b00a/774cc362-9cfe-4197-8571-7d1b1ef33e48"
 					(reference "R44")
@@
 		)
 		(instances
-			(project "esp-poe-4rl-V1"
+			(project "eumesmo-poe-4rl-v1"
 				(path "/2bc5a21a-1d79-419d-a592-6852cc07b00a/774cc362-9cfe-4197-8571-7d1b1ef33e48"
 					(reference "#PWR064")
@@
 		)
 		(instances
-			(project "esp-poe-4rl-V1"
+			(project "eumesmo-poe-4rl-v1"
 				(path "/2bc5a21a-1d79-419d-a592-6852cc07b00a/774cc362-9cfe-4197-8571-7d1b1ef33e48"
 					(reference "R47")
@@
 		)
 		(instances
-			(project "esp-poe-4rl-V1"
+			(project "eumesmo-poe-4rl-v1"
 				(path "/2bc5a21a-1d79-419d-a592-6852cc07b00a/774cc362-9cfe-4197-8571-7d1b1ef33e48"
 					(reference "D13")
@@
 		)
 		(instances
-			(project "esp-poe-4rl-V1"
+			(project "eumesmo-poe-4rl-v1"
 				(path "/2bc5a21a-1d79-419d-a592-6852cc07b00a/774cc362-9cfe-4197-8571-7d1b1ef33e48"
 					(reference "R39")
@@
 		)
 		(instances
-			(project "esp-poe-4rl-V1"
+			(project "eumesmo-poe-4rl-v1"
 				(path "/2bc5a21a-1d79-419d-a592-6852cc07b00a/774cc362-9cfe-4197-8571-7d1b1ef33e48"
 					(reference "J5")
@@
 		)
 		(instances
-			(project "esp-poe-4rl-V1"
+			(project "eumesmo-poe-4rl-v1"
 				(path "/2bc5a21a-1d79-419d-a592-6852cc07b00a/774cc362-9cfe-4197-8571-7d1b1ef33e48"
 					(reference "R48")
@@
 		)
 		(instances
-			(project "esp-poe-4rl-V1"
+			(project "eumesmo-poe-4rl-v1"
 				(path "/2bc5a21a-1d79-419d-a592-6852cc07b00a/774cc362-9cfe-4197-8571-7d1b1ef33e48"
 					(reference "J4")
@@
 		)
 		(instances
-			(project "esp-poe-4rl-V1"
+			(project "eumesmo-poe-4rl-v1"
 				(path "/2bc5a21a-1d79-419d-a592-6852cc07b00a/774cc362-9cfe-4197-8571-7d1b1ef33e48"
 					(reference "#PWR073")
@@
 		)
 		(instances
-			(project "esp-poe-4rl-V1"
+			(project "eumesmo-poe-4rl-v1"
 				(path "/2bc5a21a-1d79-419d-a592-6852cc07b00a/774cc362-9cfe-4197-8571-7d1b1ef33e48"
 					(reference "Q6")
@@
 		)
 		(instances
-			(project "esp-poe-4rl-V1"
+			(project "eumesmo-poe-4rl-v1"
 				(path "/2bc5a21a-1d79-419d-a592-6852cc07b00a/774cc362-9cfe-4197-8571-7d1b1ef33e48"
 					(reference "#PWR075")
@@
 		)
 		(instances
-			(project "esp-poe-4rl-V1"
+			(project "eumesmo-poe-4rl-v1"
 				(path "/2bc5a21a-1d79-419d-a592-6852cc07b00a/774cc362-9cfe-4197-8571-7d1b1ef33e48"
 					(reference "#PWR070")
@@
 		)
 		(instances
-			(project "esp-poe-4rl-V1"
+			(project "eumesmo-poe-4rl-v1"
 				(path "/2bc5a21a-1d79-419d-a592-6852cc07b00a/774cc362-9cfe-4197-8571-7d1b1ef33e48"
 					(reference "K1")
@@
 		)
 		(instances
-			(project "esp-poe-4rl-V1"
+			(project "eumesmo-poe-4rl-v1"
 				(path "/2bc5a21a-1d79-419d-a592-6852cc07b00a/774cc362-9cfe-4197-8571-7d1b1ef33e48"
 					(reference "D9")
@@
 		)
 		(instances
-			(project "esp-poe-4rl-V1"
+			(project "eumesmo-poe-4rl-v1"
 				(path "/2bc5a21a-1d79-419d-a592-6852cc07b00a/774cc362-9cfe-4197-8571-7d1b1ef33e48"
 					(reference "R45")
@@
 		)
 		(instances
-			(project "esp-poe-4rl-V1"
+			(project "eumesmo-poe-4rl-v1"
 				(path "/2bc5a21a-1d79-419d-a592-6852cc07b00a/774cc362-9cfe-4197-8571-7d1b1ef33e48"
 					(reference "J3")
@@
 		)
 		(instances
-			(project "esp-poe-4rl-V1"
+			(project "eumesmo-poe-4rl-v1"
 				(path "/2bc5a21a-1d79-419d-a592-6852cc07b00a/774cc362-9cfe-4197-8571-7d1b1ef33e48"
 					(reference "#PWR068")
@@
 		)
 		(instances
-			(project "esp-poe-4rl-V1"
+			(project "eumesmo-poe-4rl-v1"
 				(path "/2bc5a21a-1d79-419d-a592-6852cc07b00a/774cc362-9cfe-4197-8571-7d1b1ef33e48"
 					(reference "R40")
@@
 		)
 		(instances
-			(project "esp-poe-4rl-V1"
+			(project "eumesmo-poe-4rl-v1"
 				(path "/2bc5a21a-1d79-419d-a592-6852cc07b00a/774cc362-9cfe-4197-8571-7d1b1ef33e48"
 					(reference "#PWR066")
@@
 		)
 		(instances
-			(project "esp-poe-4rl-V1"
+			(project "eumesmo-poe-4rl-v1"
 				(path "/2bc5a21a-1d79-419d-a592-6852cc07b00a/774cc362-9cfe-4197-8571-7d1b1ef33e48"
 					(reference "K3")
@@
 		)
 		(instances
-			(project "esp-poe-4rl-V1"
+			(project "eumesmo-poe-4rl-v1"
 				(path "/2bc5a21a-1d79-419d-a592-6852cc07b00a/774cc362-9cfe-4197-8571-7d1b1ef33e48"
 					(reference "#PWR072")
@@
 		)
 		(instances
-			(project "esp-poe-4rl-V1"
+			(project "eumesmo-poe-4rl-v1"
 				(path "/2bc5a21a-1d79-419d-a592-6852cc07b00a/774cc362-9cfe-4197-8571-7d1b1ef33e48"
 					(reference "Q4")
@@
 		)
 		(instances
-			(project "esp-poe-4rl-V1"
+			(project "eumesmo-poe-4rl-v1"
 				(path "/2bc5a21a-1d79-419d-a592-6852cc07b00a/774cc362-9cfe-4197-8571-7d1b1ef33e48"
 					(reference "Q5")
@@
 		)
 		(instances
-			(project "esp-poe-4rl-V1"
+			(project "eumesmo-poe-4rl-v1"
 				(path "/2bc5a21a-1d79-419d-a592-6852cc07b00a/774cc362-9cfe-4197-8571-7d1b1ef33e48"
 					(reference "#PWR071")
@@
 		)
 		(instances
-			(project "esp-poe-4rl-V1"
+			(project "eumesmo-poe-4rl-v1"
 				(path "/2bc5a21a-1d79-419d-a592-6852cc07b00a/774cc362-9cfe-4197-8571-7d1b1ef33e48"
 					(reference "Q7")
@@
 		)
 		(instances
-			(project "esp-poe-4rl-V1"
+			(project "eumesmo-poe-4rl-v1"
 				(path "/2bc5a21a-1d79-419d-a592-6852cc07b00a/774cc362-9cfe-4197-8571-7d1b1ef33e48"
 					(reference "J6")
@@
 		)
 		(instances
-			(project "esp-poe-4rl-V1"
+			(project "eumesmo-poe-4rl-v1"
 				(path "/2bc5a21a-1d79-419d-a592-6852cc07b00a/774cc362-9cfe-4197-8571-7d1b1ef33e48"
 					(reference "#PWR069")
@@
 		)
 		(instances
-			(project "esp-poe-4rl-V1"
+			(project "eumesmo-poe-4rl-v1"
 				(path "/2bc5a21a-1d79-419d-a592-6852cc07b00a/774cc362-9cfe-4197-8571-7d1b1ef33e48"
 					(reference "R46")
@@
 		)
 		(instances
-			(project "esp-poe-4rl-V1"
+			(project "eumesmo-poe-4rl-v1"
 				(path "/2bc5a21a-1d79-419d-a592-6852cc07b00a/774cc362-9cfe-4197-8571-7d1b1ef33e48"
 					(reference "#PWR067")
@@
 		)
 		(instances
-			(project "esp-poe-4rl-V1"
+			(project "eumesmo-poe-4rl-v1"
 				(path "/2bc5a21a-1d79-419d-a592-6852cc07b00a/774cc362-9cfe-4197-8571-7d1b1ef33e48"
 					(reference "D14")

Commit message: Added CPU health LED
Parts:
- renumbered D9 to D10, D10 to D11, D11 to D12, D12 to D13, D13 to D14, D14 to D15, D15 to D16, D8 to D9, R38 to R39, R39 to R40, R40 to R41, R41 to R42, R42 to R43, R43 to R44, R44 to R45, R45 to R46, R46 to R47, R47 to R48, R48 to R49, R49 to R50
