File: V1/eumesmo-poe-4rl-v1-outputs.kicad_sch (KiCad schematic)
At the start: 32 parts, among them J3 250-202, J4 250-202, J5 250-202, J6 250-202, K1 G5NB-1A-E-DC5, K2 G5NB-1A-E-DC5, K3 G5NB-1A-E-DC5, K4 G5NB-1A-E-DC5, Q4 MMBT2222A, Q5 MMBT2222A, Q6 MMBT2222A, Q7 MMBT2222A

Commit message: Adjusted components according to availability in JLCPCB.
Parts:
- D11, D12, D15, D16: value WHITE -> WHITE/0603
- R39, R40, R45, R46: value 680R -> 1k; LCSC Part # C25130 -> C11702; Mfr PN 0402WGF6800TCE -> 0402WGF1001TCE; Vendor PN C25130 -> C11702
Other:
- note added: "I_{LED} = (5V - V_{LED} - V_{CE}) / 1k I_{LED} = (5V - 2.7V - 0,1V) / 1k I_{LED} = 2,3 mA"
Changed lines of the file:
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@@
 		(rev "V1.1")
 	)
+	(text "I_{LED} = (5V - V_{LED} - V_{CE}) / 1k\nI_{LED} = (5V - 2.7V - 0,1V) / 1k\nI_{LED} = 2,3 mA"
+		(exclude_from_sim no)
+		(at 68.58 40.64 0)
+		(effects
+			(font
+				(size 1.5 1.5)
+			)
+			(justify left bottom)
+		)
+	)
 	(junction
 		(at 81.28 49.53)
@@
 			)
 		)
-		(property "Value" "680R"
+		(property "Value" "1k"
 			(at 64.77 55.8799 0)
 			(show_name no)
@@
 			)
 		)
-		(property "Mfr PN" "0402WGF6800TCE"
+		(property "Mfr PN" "0402WGF1001TCE"
 			(at 62.23 55.88 0)
 			(hide yes)
@@
 			)
 		)
-		(property "Vendor PN" "C25130"
+		(property "Vendor PN" "C11702"
 			(at 62.23 55.88 0)
 			(hide yes)
@@
 			)
 		)
-		(property "LCSC Part #" "C25130"
+		(property "LCSC Part #" "C11702"
 			(at 64.77 58.4199 0)
 			(show_name no)
@@
 			)
 		)
-		(property "Value" "WHITE"
+		(property "Value" "WHITE/0603"
 			(at 64.77 65.9764 90)
 			(show_name no)
@@
 			)
 		)
-		(property "Value" "WHITE"
+		(property "Value" "WHITE/0603"
 			(at 193.04 65.9764 90)
 			(show_name no)
@@
 			)
 		)
-		(property "Value" "WHITE"
+		(property "Value" "WHITE/0603"
 			(at 193.04 110.4264 90)
 			(show_name no)
@@
 			)
 		)
-		(property "Value" "680R"
+		(property "Value" "1k"
 			(at 64.77 100.3299 0)
 			(show_name no)
@@
 			)
 		)
-		(property "Mfr PN" "0402WGF6800TCE"
+		(property "Mfr PN" "0402WGF1001TCE"
 			(at 62.23 100.33 0)
 			(hide yes)
@@
 			)
 		)
-		(property "Vendor PN" "C25130"
+		(property "Vendor PN" "C11702"
 			(at 62.23 100.33 0)
 			(hide yes)
@@
 			)
 		)
-		(property "LCSC Part #" "C25130"
+		(property "LCSC Part #" "C11702"
 			(at 64.77 102.8699 0)
 			(show_name no)
@@
 			)
 		)
-		(property "Value" "680R"
+		(property "Value" "1k"
 			(at 193.04 55.8799 0)
 			(show_name no)
@@
 			)
 		)
-		(property "Mfr PN" "0402WGF6800TCE"
+		(property "Mfr PN" "0402WGF1001TCE"
 			(at 190.5 55.88 0)
 			(hide yes)
@@
 			)
 		)
-		(property "Vendor PN" "C25130"
+		(property "Vendor PN" "C11702"
 			(at 190.5 55.88 0)
 			(hide yes)
@@
 			)
 		)
-		(property "LCSC Part #" "C25130"
+		(property "LCSC Part #" "C11702"
 			(at 193.04 58.4199 0)
 			(show_name no)
@@
 			)
 		)
-		(property "Value" "680R"
+		(property "Value" "1k"
 			(at 193.04 100.3299 0)
 			(show_name no)
@@
 			)
 		)
-		(property "Mfr PN" "0402WGF6800TCE"
+		(property "Mfr PN" "0402WGF1001TCE"
 			(at 190.5 100.33 0)
 			(hide yes)
@@
 			)
 		)
-		(property "Vendor PN" "C25130"
+		(property "Vendor PN" "C11702"
 			(at 190.5 100.33 0)
 			(hide yes)
@@
 			)
 		)
-		(property "LCSC Part #" "C25130"
+		(property "LCSC Part #" "C11702"
 			(at 193.04 102.8699 0)
 			(show_name no)
@@
 			)
 		)
-		(property "Value" "WHITE"
+		(property "Value" "WHITE/0603"
 			(at 64.77 110.4264 90)
 			(show_name no)

Commit message: LEDs replaced for orange
Parts:
- D11, D12, D15, D16: value WHITE/0603 -> ORANGE/0603; LCSC Part # C2290 -> C2987557; Mfr Hubei KENTO Elec -> Everlight Elec; Mfr PN KT-0603W -> 19-217/S2C-AL1M2VY/6T; Technology InGaN -> LED; Vendor PN C2290 -> C2987557
- R39, R40, R45, R46: value 1k -> 1.2k; LCSC Part # C11702 -> C25862; Mfr PN 0402WGF1001TCE -> 0402WGF1201TCE; Vendor PN C11702 -> C25862
Other:
- note added: "V_{F} = 1,8V @ 2,5mA I_{LED} = (5V - V_{F} - V_{CE}) / R I_{LED} = (5V - 1.8V - 0,1V) / 1.2k I_{LED} = 2,58 mA"
- note removed: "I_{LED} = (5V - V_{LED} - V_{CE}) / 1k I_{LED} = (5V - 2.7V - 0,1V) / 1k I_{LED} = 2,3 mA"
Changed lines of the file:
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@@
 		(rev "V1.1")
 	)
-	(text "I_{LED} = (5V - V_{LED} - V_{CE}) / 1k\nI_{LED} = (5V - 2.7V - 0,1V) / 1k\nI_{LED} = 2,3 mA"
+	(text "V_{F} = 1,8V @ 2,5mA\nI_{LED} = (5V - V_{F} - V_{CE}) / R\nI_{LED} = (5V - 1.8V - 0,1V) / 1.2k\nI_{LED} = 2,58 mA"
 		(exclude_from_sim no)
 		(at 68.58 40.64 0)
@@
 			)
 		)
-		(property "Value" "1k"
+		(property "Value" "1.2k"
 			(at 64.77 55.8799 0)
 			(show_name no)
@@
 			)
 		)
-		(property "Mfr PN" "0402WGF1001TCE"
+		(property "Mfr PN" "0402WGF1201TCE"
 			(at 62.23 55.88 0)
 			(hide yes)
@@
 			)
 		)
-		(property "Vendor PN" "C11702"
+		(property "Vendor PN" "C25862"
 			(at 62.23 55.88 0)
 			(hide yes)
@@
 			)
 		)
-		(property "LCSC Part #" "C11702"
+		(property "LCSC Part #" "C25862"
 			(at 64.77 58.4199 0)
 			(show_name no)
@@
 			)
 		)
-		(property "Value" "WHITE/0603"
+		(property "Value" "ORANGE/0603"
 			(at 64.77 65.9764 90)
 			(show_name no)
@@
 			)
 		)
-		(property "Mfr" "Hubei KENTO Elec"
+		(property "Mfr" "Everlight Elec"
 			(at 62.23 66.04 0)
 			(hide yes)
@@
 			)
 		)
-		(property "Mfr PN" "KT-0603W"
+		(property "Mfr PN" "19-217/S2C-AL1M2VY/6T"
 			(at 62.23 66.04 0)
 			(hide yes)
@@
 			)
 		)
-		(property "Technology" "InGaN"
+		(property "Technology" "LED"
 			(at 62.23 66.04 0)
 			(hide yes)
@@
 			)
 		)
-		(property "Vendor PN" "C2290"
+		(property "Vendor PN" "C2987557"
 			(at 62.23 66.04 0)
 			(hide yes)
@@
 			)
 		)
-		(property "LCSC Part #" "C2290"
+		(property "LCSC Part #" "C2987557"
 			(at 64.77 68.5164 90)
 			(show_name no)
@@
 			)
 		)
-		(property "Value" "WHITE/0603"
+		(property "Value" "ORANGE/0603"
 			(at 193.04 65.9764 90)
 			(show_name no)
@@
 			)
 		)
-		(property "Mfr" "Hubei KENTO Elec"
+		(property "Mfr" "Everlight Elec"
 			(at 190.5 66.04 0)
 			(hide yes)
@@
 			)
 		)
-		(property "Mfr PN" "KT-0603W"
+		(property "Mfr PN" "19-217/S2C-AL1M2VY/6T"
 			(at 190.5 66.04 0)
 			(hide yes)
@@
 			)
 		)
-		(property "Technology" "InGaN"
+		(property "Technology" "LED"
 			(at 190.5 66.04 0)
 			(hide yes)
@@
 			)
 		)
-		(property "Vendor PN" "C2290"
+		(property "Vendor PN" "C2987557"
 			(at 190.5 66.04 0)
 			(hide yes)
@@
 			)
 		)
-		(property "LCSC Part #" "C2290"
+		(property "LCSC Part #" "C2987557"
 			(at 193.04 68.5164 90)
 			(show_name no)
@@
 			)
 		)
-		(property "Value" "WHITE/0603"
+		(property "Value" "ORANGE/0603"
 			(at 193.04 110.4264 90)
 			(show_name no)
@@
 			)
 		)
-		(property "Mfr" "Hubei KENTO Elec"
+		(property "Mfr" "Everlight Elec"
 			(at 190.5 110.49 0)
 			(hide yes)
@@
 			)
 		)
-		(property "Mfr PN" "KT-0603W"
+		(property "Mfr PN" "19-217/S2C-AL1M2VY/6T"
 			(at 190.5 110.49 0)
 			(hide yes)
@@
 			)
 		)
-		(property "Technology" "InGaN"
+		(property "Technology" "LED"
 			(at 190.5 110.49 0)
 			(hide yes)
@@
 			)
 		)
-		(property "Vendor PN" "C2290"
+		(property "Vendor PN" "C2987557"
 			(at 190.5 110.49 0)
 			(hide yes)
@@
 			)
 		)
-		(property "LCSC Part #" "C2290"
+		(property "LCSC Part #" "C2987557"
 			(at 193.04 112.9664 90)
 			(show_name no)
@@
 			)
 		)
-		(property "Value" "1k"
+		(property "Value" "1.2k"
 			(at 64.77 100.3299 0)
 			(show_name no)
@@
 			)
 		)
-		(property "Mfr PN" "0402WGF1001TCE"
+		(property "Mfr PN" "0402WGF1201TCE"
 			(at 62.23 100.33 0)
 			(hide yes)
@@
 			)
 		)
-		(property "Vendor PN" "C11702"
+		(property "Vendor PN" "C25862"
 			(at 62.23 100.33 0)
 			(hide yes)
@@
 			)
 		)
-		(property "LCSC Part #" "C11702"
+		(property "LCSC Part #" "C25862"
 			(at 64.77 102.8699 0)
 			(show_name no)
@@
 			)
 		)
-		(property "Value" "1k"
+		(property "Value" "1.2k"
 			(at 193.04 55.8799 0)
 			(show_name no)
@@
 			)
 		)
-		(property "Mfr PN" "0402WGF1001TCE"
+		(property "Mfr PN" "0402WGF1201TCE"
 			(at 190.5 55.88 0)
 			(hide yes)
@@
 			)
 		)
-		(property "Vendor PN" "C11702"
+		(property "Vendor PN" "C25862"
 			(at 190.5 55.88 0)
 			(hide yes)
@@
 			)
 		)
-		(property "LCSC Part #" "C11702"
+		(property "LCSC Part #" "C25862"
 			(at 193.04 58.4199 0)
 			(show_name no)
@@
 			)
 		)
-		(property "Value" "1k"
+		(property "Value" "1.2k"
 			(at 193.04 100.3299 0)
 			(show_name no)
@@
 			)
 		)
-		(property "Mfr PN" "0402WGF1001TCE"
+		(property "Mfr PN" "0402WGF1201TCE"
 			(at 190.5 100.33 0)
 			(hide yes)
@@
 			)
 		)
-		(property "Vendor PN" "C11702"
+		(property "Vendor PN" "C25862"
 			(at 190.5 100.33 0)
 			(hide yes)
@@
 			)
 		)
-		(property "LCSC Part #" "C11702"
+		(property "LCSC Part #" "C25862"
 			(at 193.04 102.8699 0)
 			(show_name no)
@@
 			)
 		)
-		(property "Value" "WHITE/0603"
+		(property "Value" "ORANGE/0603"
 			(at 64.77 110.4264 90)
 			(show_name no)
@@
 			)
 		)
-		(property "Mfr" "Hubei KENTO Elec"
+		(property "Mfr" "Everlight Elec"
 			(at 62.23 110.49 0)
 			(hide yes)
@@
 			)
 		)
-		(property "Mfr PN" "KT-0603W"
+		(property "Mfr PN" "19-217/S2C-AL1M2VY/6T"
 			(at 62.23 110.49 0)
 			(hide yes)
@@
 			)
 		)
-		(property "Technology" "InGaN"
+		(property "Technology" "LED"
 			(at 62.23 110.49 0)
 			(hide yes)
@@
 			)
 		)
-		(property "Vendor PN" "C2290"
+		(property "Vendor PN" "C2987557"
 			(at 62.23 110.49 0)
 			(hide yes)
@@
 			)
 		)
-		(property "LCSC Part #" "C2290"
+		(property "LCSC Part #" "C2987557"
 			(at 64.77 112.9664 90)
 			(show_name no)
