File: V1/eumesmo-poe-4rl-v1.kicad_pcb (KiCad board)
At the start: 4 copper layers, 99.5 x 45 mm, 125 parts, among them J1 USB_C_Receptacle_USB2.0, J2 RJ45 JACK, J3 250-202, J4 250-202, J5 250-202, J6 250-202, K1 G5NB-1A-E-DC5, K2 G5NB-1A-E-DC5, K3 G5NB-1A-E-DC5, K4 G5NB-1A-E-DC5, Q1 UMH3N, Q2 WPM2015-3/TR, Q3 LMUN2211LT1G, Q4 MMBT2222A, Q5 MMBT2222A, Q6 MMBT2222A, Q7 MMBT2222A, SW1 RESET, U1 CH340K, U2 ESP32-WROOM-32UE-N16, U3 LAN8710A, U4 TPS2376DDAR-H, U5 TX4138, U6 SY8089A1AAC

Commit message: Adjusted components according to availability in JLCPCB.
Parts:
- D11, D12, D15, D16, D8: value WHITE -> WHITE/0603
- R15, R37: value 300R -> 330R
- R39, R40, R45, R46: value 680R -> 1k
Changed lines of the file:
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@@
 			)
 		)
-		(property "Value" "680R"
+		(property "Value" "1k"
 			(at 0 1.17 0)
 			(layer "F.Fab")
@@
 			)
 		)
-		(property "Mfr PN" "0402WGF6800TCE"
+		(property "Mfr PN" "0402WGF1001TCE"
 			(at 0 0 180)
 			(unlocked yes)
@@
 			)
 		)
-		(property "Vendor PN" "C25130"
+		(property "Vendor PN" "C11702"
 			(at 0 0 180)
 			(unlocked yes)
@@
 			)
 		)
-		(property "LCSC Part #" "C25130"
+		(property "LCSC Part #" "C11702"
 			(at 0 0 180)
 			(unlocked yes)
@@
 			)
 		)
-		(property "Value" "680R"
+		(property "Value" "1k"
 			(at 0 1.17 0)
 			(layer "F.Fab")
@@
 			)
 		)
-		(property "Mfr PN" "0402WGF6800TCE"
+		(property "Mfr PN" "0402WGF1001TCE"
 			(at 0 0 180)
 			(unlocked yes)
@@
 			)
 		)
-		(property "Vendor PN" "C25130"
+		(property "Vendor PN" "C11702"
 			(at 0 0 180)
 			(unlocked yes)
@@
 			)
 		)
-		(property "LCSC Part #" "C25130"
+		(property "LCSC Part #" "C11702"
 			(at 0 0 180)
 			(unlocked yes)
@@
 			)
 		)
-		(property "Value" "WHITE"
+		(property "Value" "WHITE/0603"
 			(at 0 1.43 0)
 			(layer "F.Fab")
@@
 			)
 		)
-		(property "Value" "WHITE"
+		(property "Value" "WHITE/0603"
 			(at 0 1.43 0)
 			(layer "F.Fab")
@@
 			)
 		)
-		(property "Value" "680R"
+		(property "Value" "1k"
 			(at 0 1.17 0)
 			(layer "F.Fab")
@@
 			)
 		)
-		(property "Mfr PN" "0402WGF6800TCE"
+		(property "Mfr PN" "0402WGF1001TCE"
 			(at 0 0 180)
 			(unlocked yes)
@@
 			)
 		)
-		(property "Vendor PN" "C25130"
+		(property "Vendor PN" "C11702"
 			(at 0 0 180)
 			(unlocked yes)
@@
 			)
 		)
-		(property "LCSC Part #" "C25130"
+		(property "LCSC Part #" "C11702"
 			(at 0 0 180)
 			(unlocked yes)
@@
 			)
 		)
-		(property "LCSC Part #" "C161353"
+		(property "LCSC Part #" "C9196"
 			(at 10.975 224.025 0)
 			(layer "F.Fab")
@@
 			)
 		)
-		(property "Mfr" "Murata Electronics"
+		(property "Mfr" "FH"
 			(at 10.975 224.025 0)
 			(layer "F.Fab")
@@
 			)
 		)
-		(property "Mfr PN" "GR431BR7LA102KW66L"
+		(property "Mfr PN" "1206B102K202NT"
 			(at 10.975 224.025 0)
 			(layer "F.Fab")
@@
 			)
 		)
-		(property "Vendor PN" "C161353"
+		(property "Vendor PN" "C9196"
 			(at 10.975 224.025 0)
 			(layer "F.Fab")
@@
 			)
 		)
-		(property "Value" "680R"
+		(property "Value" "1k"
 			(at 0 1.17 0)
 			(layer "F.Fab")
@@
 			)
 		)
-		(property "Mfr PN" "0402WGF6800TCE"
+		(property "Mfr PN" "0402WGF1001TCE"
 			(at 0 0 180)
 			(unlocked yes)
@@
 			)
 		)
-		(property "Vendor PN" "C25130"
+		(property "Vendor PN" "C11702"
 			(at 0 0 180)
 			(unlocked yes)
@@
 			)
 		)
-		(property "LCSC Part #" "C25130"
+		(property "LCSC Part #" "C11702"
 			(at 0 0 180)
 			(unlocked yes)
@@
 			)
 		)
-		(property "LCSC Part #" "C185323"
+		(property "LCSC Part #" "C23198"
 			(at 283.35 199 0)
 			(layer "F.Fab")
@@
 			)
 		)
-		(property "Mfr" "Yageo"
+		(property "Mfr" "Uniroyal"
 			(at 283.35 199 0)
 			(layer "F.Fab")
@@
 			)
 		)
-		(property "Mfr PN" "RC0603FR-0752K3L"
+		(property "Mfr PN" "0603WAF5232T5E"
 			(at 283.35 199 0)
 			(layer "F.Fab")
@@
 			)
 		)
-		(property "Vendor PN" "C185323"
+		(property "Vendor PN" "C23198"
 			(at 283.35 199 0)
 			(layer "F.Fab")
@@
 			)
 		)
-		(property "Value" "300R"
+		(property "Value" "330R"
 			(at 0 1.17 90)
 			(layer "F.Fab")
@@
 			)
 		)
-		(property "Mfr PN" "0402WGF3000TCE"
+		(property "Mfr PN" "0402WGF3300TCE"
 			(at 0 0 270)
 			(unlocked yes)
@@
 			)
 		)
-		(property "Vendor PN" "C25102"
+		(property "Vendor PN" "C25104"
 			(at 0 0 270)
 			(unlocked yes)
@@
 			)
 		)
-		(property "LCSC Part #" "C25102"
+		(property "LCSC Part #" "C25104"
 			(at 0 0 270)
 			(unlocked yes)
@@
 			)
 		)
+		(property "Package" "0402/1005"
+			(at 0 0 270)
+			(unlocked yes)
+			(layer "F.Fab")
+			(hide yes)
+			(effects
+				(font
+					(size 1 1)
+					(thickness 0.15)
+				)
+			)
+		)
 		(property ki_fp_filters "R_*")
 		(sheetname "/")
@@
 			)
 		)
-		(property "Value" "WHITE"
+		(property "Value" "WHITE/0603"
 			(at 0 1.43 0)
 			(layer "F.Fab")
@@
 			)
 		)
-		(property "Value" "WHITE"
+		(property "Value" "WHITE/0603"
 			(at 0 1.43 0)
 			(layer "F.Fab")
@@
 			)
 		)
-		(property "Value" "WHITE"
+		(property "Value" "WHITE/0603"
 			(at 0 1.43 90)
 			(layer "F.Fab")
@@
 			)
 		)
-		(property "Value" "300R"
+		(property "Value" "330R"
 			(at 0 1.17 0)
 			(layer "F.Fab")
@@
 			)
 		)
-		(property "Mfr PN" "0402WGF3000TCE"
+		(property "Mfr PN" "0402WGF3300TCE"
 			(at 0 0 0)
 			(unlocked yes)
@@
 			)
 		)
-		(property "Vendor PN" "C25102"
+		(property "Vendor PN" "C25104"
 			(at 0 0 0)
 			(unlocked yes)
@@
 			)
 		)
-		(property "LCSC Part #" "C25102"
+		(property "LCSC Part #" "C25104"
 			(at 0 0 0)
 			(unlocked yes)
