File: V1/eumesmo-poe-4rl-v1-power.kicad_sch (KiCad schematic)
At the start: 31 parts, among them U4 TPS2376DDAR-H, U5 TX4138, U6 SY8089A1AAC

Commit message: Adjusted components according to availability in JLCPCB.
Parts:
- D8: value WHITE -> WHITE/0603
- R35: LCSC Part # C185323 -> C23198; Mfr Yageo -> Uniroyal; Mfr PN RC0603FR-0752K3L -> 0603WAF5232T5E; Vendor PN C185323 -> C23198
- R37: value 300R -> 330R; LCSC Part # C25102 -> C25104; Mfr PN 0402WGF3000TCE -> 0402WGF3300TCE; Vendor PN C25102 -> C25104
Changed lines of the file:
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@@
 			)
 		)
-		(property "Value" "WHITE"
+		(property "Value" "WHITE/0603"
 			(at 133.35 170.1164 90)
 			(show_name no)
@@
 			)
 		)
-		(property "LCSC Part #" "C185323"
+		(property "LCSC Part #" "C23198"
 			(at 137.16 125.7299 0)
 			(show_name no)
@@
 			)
 		)
-		(property "Mfr" "Yageo"
+		(property "Mfr" "Uniroyal"
 			(at 134.62 123.19 0)
 			(hide yes)
@@
 			)
 		)
-		(property "Mfr PN" "RC0603FR-0752K3L"
+		(property "Mfr PN" "0603WAF5232T5E"
 			(at 134.62 123.19 0)
 			(hide yes)
@@
 			)
 		)
-		(property "Vendor PN" "C185323"
+		(property "Vendor PN" "C23198"
 			(at 134.62 123.19 0)
 			(hide yes)
@@
 			)
 		)
-		(property "Value" "300R"
+		(property "Value" "330R"
 			(at 133.35 156.2099 0)
 			(show_name no)
@@
 			)
 		)
-		(property "Mfr PN" "0402WGF3000TCE"
+		(property "Mfr PN" "0402WGF3300TCE"
 			(at 130.81 156.21 0)
 			(hide yes)
@@
 			)
 		)
-		(property "Vendor PN" "C25102"
+		(property "Vendor PN" "C25104"
 			(at 130.81 156.21 0)
 			(hide yes)
@@
 			)
 		)
-		(property "LCSC Part #" "C25102"
+		(property "LCSC Part #" "C25104"
 			(at 133.35 158.7499 0)
 			(show_name no)

Commit message: LEDs replaced for orange
Parts:
- D8: value WHITE/0603 -> ORANGE/0603; LCSC Part # C2290 -> C2987557; Mfr Hubei KENTO Elec -> Everlight Elec; Mfr PN KT-0603W -> 19-217/S2C-AL1M2VY/6T; Technology InGaN -> LED; Vendor PN C2290 -> C2987557
- R37: value 330R -> 680R; LCSC Part # C25104 -> C25130; Mfr PN 0402WGF3300TCE -> 0402WGF6800TCE; Vendor PN C25104 -> C25130
Other:
- note added: "V_{F} = 1,8V @ 2,5mA I_{LED} = (3.3V - V_{F}) / R I_{LED} = (3.3V - 1.8V) / 680R I_{LED} = 2,20 mA"
Changed lines of the file:
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@@
 		)
 	)
+	(text "V_{F} = 1,8V @ 2,5mA\nI_{LED} = (3.3V - V_{F}) / R\nI_{LED} = (3.3V - 1.8V) / 680R\nI_{LED} = 2,20 mA"
+		(exclude_from_sim no)
+		(at 129.54 190.5 0)
+		(effects
+			(font
+				(size 1.5 1.5)
+			)
+			(justify left bottom)
+		)
+	)
 	(text "R_{TX1}"
 		(exclude_from_sim no)
@@
 			)
 		)
-		(property "Value" "WHITE/0603"
+		(property "Value" "ORANGE/0603"
 			(at 133.35 170.1164 90)
 			(show_name no)
@@
 			)
 		)
-		(property "Mfr" "Hubei KENTO Elec"
+		(property "Mfr" "Everlight Elec"
 			(at 130.81 170.18 0)
 			(hide yes)
@@
 			)
 		)
-		(property "Mfr PN" "KT-0603W"
+		(property "Mfr PN" "19-217/S2C-AL1M2VY/6T"
 			(at 130.81 170.18 0)
 			(hide yes)
@@
 			)
 		)
-		(property "Technology" "InGaN"
+		(property "Technology" "LED"
 			(at 130.81 170.18 0)
 			(hide yes)
@@
 			)
 		)
-		(property "Vendor PN" "C2290"
+		(property "Vendor PN" "C2987557"
 			(at 130.81 170.18 0)
 			(hide yes)
@@
 			)
 		)
-		(property "LCSC Part #" "C2290"
+		(property "LCSC Part #" "C2987557"
 			(at 133.35 172.6564 90)
 			(show_name no)
@@
 			)
 		)
-		(property "Value" "330R"
+		(property "Value" "680R"
 			(at 133.35 156.2099 0)
 			(show_name no)
@@
 			)
 		)
-		(property "Mfr PN" "0402WGF3300TCE"
+		(property "Mfr PN" "0402WGF6800TCE"
 			(at 130.81 156.21 0)
 			(hide yes)
@@
 			)
 		)
-		(property "Vendor PN" "C25104"
+		(property "Vendor PN" "C25130"
 			(at 130.81 156.21 0)
 			(hide yes)
@@
 			)
 		)
-		(property "LCSC Part #" "C25104"
+		(property "LCSC Part #" "C25130"
 			(at 133.35 158.7499 0)
 			(show_name no)
