File: V1/eumesmo-poe-4rl-v1.kicad_sch (KiCad schematic)
At the start: 58 parts, among them J1 USB_C_Receptacle_USB2.0, J2 RJ45 JACK, Q1 UMH3N, Q2 WPM2015-3/TR, Q3 LMUN2211LT1G, SW1 RESET, U1 CH340K, U2 ESP32-WROOM-32UE-N16, U3 LAN8710A

Commit message: LEDs replaced for orange
Parts:
- D3: value WHITE/0603 -> ORANGE/0603; LCSC Part # C2290 -> C2987557; Mfr Hubei KENTO Elec -> Everlight Elec; Mfr PN KT-0603W -> 19-217/S2C-AL1M2VY/6T; Package (none) -> 0603/1608; Vendor PN C2290 -> C2987557
- R15: value 330R -> 680R; LCSC Part # C25104 -> C25130; Mfr PN 0402WGF3300TCE -> 0402WGF6800TCE; Vendor PN C25104 -> C25130
Changed lines of the file:
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@@
 			)
 		)
-		(property "Value" "330R"
+		(property "Value" "680R"
 			(at 232.41 119.38 90)
 			(show_name no)
@@
 			)
 		)
-		(property "Mfr PN" "0402WGF3300TCE"
+		(property "Mfr PN" "0402WGF6800TCE"
 			(at 232.41 125.73 0)
 			(hide yes)
@@
 			)
 		)
-		(property "Vendor PN" "C25104"
+		(property "Vendor PN" "C25130"
 			(at 232.41 125.73 0)
 			(hide yes)
@@
 			)
 		)
-		(property "LCSC Part #" "C25104"
+		(property "LCSC Part #" "C25130"
 			(at 232.41 121.92 90)
 			(show_name no)
@@
 			)
 		)
-		(property "Value" "WHITE/0603"
+		(property "Value" "ORANGE/0603"
 			(at 250.1265 119.38 0)
 			(show_name no)
@@
 			)
 		)
-		(property "Mfr" "Hubei KENTO Elec"
+		(property "Mfr" "Everlight Elec"
 			(at 250.19 125.73 0)
 			(hide yes)
@@
 			)
 		)
-		(property "Mfr PN" "KT-0603W"
+		(property "Mfr PN" "19-217/S2C-AL1M2VY/6T"
 			(at 250.19 125.73 0)
 			(hide yes)
@@
 			)
 		)
-		(property "Vendor PN" "C2290"
+		(property "Vendor PN" "C2987557"
 			(at 250.19 125.73 0)
 			(hide yes)
@@
 			)
 		)
-		(property "LCSC Part #" "C2290"
+		(property "LCSC Part #" "C2987557"
 			(at 250.1265 121.92 0)
 			(show_name no)
@@
 			(at 250.19 125.73 0)
 			(hide yes)
+			(show_name no)
+			(do_not_autoplace no)
+			(effects
+				(font
+					(size 1.27 1.27)
+				)
+			)
+		)
+		(property "Package" "0603/1608"
+			(at 250.19 125.73 0)
+			(hide yes)
